Commit message: can be run

File: urdf/robot_model_gazebo.xacro (robot description, xacro)
@@ -7,19 +7,19 @@
 	<!-- KINECT ATTACHMENT -->
 	<xacro:include filename="$(find robot_model_gazebo)/urdf/sensors/kinect.xacro"/>
-	<kinect_sensor parent="kinect_base_link">
+	<xacro:kinect_sensor parent="kinect_base_link">
 		<!--origin xyz="0 0 0" rpy="0 0 0" /-->
-	</kinect_sensor>
+	</xacro:kinect_sensor>
 	<!-- LASER ATTACHMENT -->
 	<xacro:include filename="$(find robot_model_gazebo)/urdf/sensors/hokuyo.xacro"/>
-	<hokuyo_sensor parent="upper_base_link">
+	<xacro:hokuyo_sensor parent="upper_base_link">
 		<!--origin xyz="0 0 0" rpy="0 0 0" /-->
-	</hokuyo_sensor>
+	</xacro:hokuyo_sensor>
 	<!-- Import all Gazebo-customization elements, including Gazebo colors, sensors, controller -->
   	<xacro:include filename="$(find robot_model_gazebo)/urdf/robot_model_gazebo.gazebo" />
 	<!-- Add view camera - working -->
 	<xacro:include filename="$(find robot_model_gazebo)/urdf/sensors/view_camera.xacro" />
-	<view_camera_sensor parent="kinect_base_link">
+	<xacro:view_camera_sensor parent="kinect_base_link">
 		<!--origin xyz="0 0 0" rpy="0 0 0" /-->
-	</view_camera_sensor>
+	</xacro:view_camera_sensor>
 	<xacro:property name="length_wheel" value="0.075" />
 	<xacro:property name="radius_wheel" value="0.0775" />

File: urdf/sensors/kinect.xacro (robot description, xacro)
@@ -3,4 +3,11 @@
   <xacro:include filename="$(find robot_model_gazebo)/urdf/sensors/kinect_gazebo.xacro"/>
   <xacro:include filename="$(find robot_model_gazebo)/urdf/sensors/kinect_properties.xacro"/>
+  <xacro:property name="M_PI" value="3.1415926535897932384626433832795 " />
+	<xacro:property name="cam_px" value="0.028" />
+	<xacro:property name="cam_py" value="-0.0125" />
+	<xacro:property name="cam_pz" value="0.075" />
+	<xacro:property name="cam_or" value="0" />
+	<xacro:property name="cam_op" value="0" />
+	<xacro:property name="cam_oy" value="0" />
   <!-- Kinect driver in kinect_gazebo.xacro -->
   <!-- Parameterised in part by the values in kinect_properties.xacro -->
